File: Display_Driver.kicad_sch (KiCad schematic)
At the start: 80 parts, among them Q1 MPSA42, Q10 MPSA42, Q11 MPSA42, Q12 MPSA42, Q13 KSP92BU, Q14 KSP92BU, Q15 MPSA42, Q16 MPSA42, Q17 MPSA42, Q18 MPSA42, Q19 KSP92BU, Q2 MPSA42, Q20 KSP92BU, Q21 MPSA42, Q22 MPSA42, Q23 KSP92BU, Q24 KSP92BU, Q3 MPSA42, Q4 MPSA42, Q5 MPSA42, Q6 MPSA42, Q7 MPSA42, Q8 MPSA42, Q9 MPSA42

Commit message: layout started
Parts:
- Q1, Q10, Q11, Q12, Q13, Q14, Q15, Q16, Q17, Q18, Q19, Q2, Q20, Q21, Q22, Q23, Q24, Q3, Q4, Q5, Q6, Q7, Q8, Q9: footprint Package_TO_SOT_THT:TO-92_Inline -> Package_TO_SOT_THT:TO-92_Inline_Wide
Changed lines of the file:
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@@
       (effects (font (size 1.27 1.27)) (justify left))
     )
-    (property "Footprint" "Package_TO_SOT_THT:TO-92_Inline" (id 2) (at 49.53 84.455 0)
+    (property "Footprint" "Package_TO_SOT_THT:TO-92_Inline_Wide" (id 2) (at 49.53 84.455 0)
       (effects (font (size 1.27 1.27) italic) (justify left) hide)
     )
@@
       (effects (font (size 1.27 1.27)) (justify left))
     )
-    (property "Footprint" "Package_TO_SOT_THT:TO-92_Inline" (id 2) (at 74.93 84.455 0)
+    (property "Footprint" "Package_TO_SOT_THT:TO-92_Inline_Wide" (id 2) (at 74.93 84.455 0)
       (effects (font (size 1.27 1.27) italic) (justify left) hide)
     )
@@
       (effects (font (size 1.27 1.27)) (justify left))
     )
-    (property "Footprint" "Package_TO_SOT_THT:TO-92_Inline" (id 2) (at 129.54 47.625 0)
+    (property "Footprint" "Package_TO_SOT_THT:TO-92_Inline_Wide" (id 2) (at 129.54 47.625 0)
       (effects (font (size 1.27 1.27) italic) (justify left) hide)
     )
@@
       (effects (font (size 1.27 1.27)) (justify left))
     )
-    (property "Footprint" "Package_TO_SOT_THT:TO-92_Inline" (id 2) (at 129.54 98.425 0)
+    (property "Footprint" "Package_TO_SOT_THT:TO-92_Inline_Wide" (id 2) (at 129.54 98.425 0)
       (effects (font (size 1.27 1.27) italic) (justify left) hide)
     )
@@
       (effects (font (size 1.27 1.27)) (justify left))
     )
-    (property "Footprint" "Package_TO_SOT_THT:TO-92_Inline" (id 2) (at 189.23 98.425 0)
+    (property "Footprint" "Package_TO_SOT_THT:TO-92_Inline_Wide" (id 2) (at 189.23 98.425 0)
       (effects (font (size 1.27 1.27) italic) (justify left) hide)
     )
@@
       (effects (font (size 1.27 1.27)) (justify left))
     )
-    (property "Footprint" "Package_TO_SOT_THT:TO-92_Inline" (id 2) (at 189.23 47.625 0)
+    (property "Footprint" "Package_TO_SOT_THT:TO-92_Inline_Wide" (id 2) (at 189.23 47.625 0)
       (effects (font (size 1.27 1.27) italic) (justify left) hide)
     )
@@
       (effects (font (size 1.27 1.27)) (justify left))
     )
-    (property "Footprint" "Package_TO_SOT_THT:TO-92_Inline" (id 2) (at 250.19 47.625 0)
+    (property "Footprint" "Package_TO_SOT_THT:TO-92_Inline_Wide" (id 2) (at 250.19 47.625 0)
       (effects (font (size 1.27 1.27) italic) (justify left) hide)
     )
@@
       (effects (font (size 1.27 1.27)) (justify left))
     )
-    (property "Footprint" "Package_TO_SOT_THT:TO-92_Inline" (id 2) (at 250.19 98.425 0)
+    (property "Footprint" "Package_TO_SOT_THT:TO-92_Inline_Wide" (id 2) (at 250.19 98.425 0)
       (effects (font (size 1.27 1.27) italic) (justify left) hide)
     )
@@
       (effects (font (size 1.27 1.27)) (justify left))
     )
-    (property "Footprint" "Package_TO_SOT_THT:TO-92_Inline" (id 2) (at 38.1 136.525 0)
+    (property "Footprint" "Package_TO_SOT_THT:TO-92_Inline_Wide" (id 2) (at 38.1 136.525 0)
       (effects (font (size 1.27 1.27) italic) (justify left) hide)
     )
@@
       (effects (font (size 1.27 1.27)) (justify left))
     )
-    (property "Footprint" "Package_TO_SOT_THT:TO-92_Inline" (id 2) (at 69.85 136.525 0)
+    (property "Footprint" "Package_TO_SOT_THT:TO-92_Inline_Wide" (id 2) (at 69.85 136.525 0)
       (effects (font (size 1.27 1.27) italic) (justify left) hide)
     )
@@
       (effects (font (size 1.27 1.27)) (justify left))
     )
-    (property "Footprint" "Package_TO_SOT_THT:TO-92_Inline" (id 2) (at 101.6 136.525 0)
+    (property "Footprint" "Package_TO_SOT_THT:TO-92_Inline_Wide" (id 2) (at 101.6 136.525 0)
       (effects (font (size 1.27 1.27) italic) (justify left) hide)
     )
@@
       (effects (font (size 1.27 1.27)) (justify left))
     )
-    (property "Footprint" "Package_TO_SOT_THT:TO-92_Inline" (id 2) (at 133.35 136.525 0)
+    (property "Footprint" "Package_TO_SOT_THT:TO-92_Inline_Wide" (id 2) (at 133.35 136.525 0)
       (effects (font (size 1.27 1.27) italic) (justify left) hide)
     )
@@
       (effects (font (size 1.27 1.27)) (justify left))
     )
-    (property "Footprint" "Package_TO_SOT_THT:TO-92_Inline" (id 2) (at 165.1 136.525 0)
+    (property "Footprint" "Package_TO_SOT_THT:TO-92_Inline_Wide" (id 2) (at 165.1 136.525 0)
       (effects (font (size 1.27 1.27) italic) (justify left) hide)
     )
@@
       (effects (font (size 1.27 1.27)) (justify left))
     )
-    (property "Footprint" "Package_TO_SOT_THT:TO-92_Inline" (id 2) (at 165.1 175.895 0)
+    (property "Footprint" "Package_TO_SOT_THT:TO-92_Inline_Wide" (id 2) (at 165.1 175.895 0)
       (effects (font (size 1.27 1.27) italic) (justify left) hide)
     )
@@
       (effects (font (size 1.27 1.27)) (justify left))
     )
-    (property "Footprint" "Package_TO_SOT_THT:TO-92_Inline" (id 2) (at 133.35 175.895 0)
+    (property "Footprint" "Package_TO_SOT_THT:TO-92_Inline_Wide" (id 2) (at 133.35 175.895 0)
       (effects (font (size 1.27 1.27) italic) (justify left) hide)
     )
@@
       (effects (font (size 1.27 1.27)) (justify left))
     )
-    (property "Footprint" "Package_TO_SOT_THT:TO-92_Inline" (id 2) (at 101.6 175.895 0)
+    (property "Footprint" "Package_TO_SOT_THT:TO-92_Inline_Wide" (id 2) (at 101.6 175.895 0)
       (effects (font (size 1.27 1.27) italic) (justify left) hide)
     )
@@
       (effects (font (size 1.27 1.27)) (justify left))
     )
-    (property "Footprint" "Package_TO_SOT_THT:TO-92_Inline" (id 2) (at 69.85 175.895 0)
+    (property "Footprint" "Package_TO_SOT_THT:TO-92_Inline_Wide" (id 2) (at 69.85 175.895 0)
       (effects (font (size 1.27 1.27) italic) (justify left) hide)
     )
@@
       (effects (font (size 1.27 1.27)) (justify left))
     )
-    (property "Footprint" "Package_TO_SOT_THT:TO-92_Inline" (id 2) (at 38.1 175.895 0)
+    (property "Footprint" "Package_TO_SOT_THT:TO-92_Inline_Wide" (id 2) (at 38.1 175.895 0)
       (effects (font (size 1.27 1.27) italic) (justify left) hide)
     )
@@
       (effects (font (size 1.27 1.27)) (justify left))
     )
-    (property "Footprint" "Package_TO_SOT_THT:TO-92_Inline" (id 2) (at 142.24 28.575 0)
+    (property "Footprint" "Package_TO_SOT_THT:TO-92_Inline_Wide" (id 2) (at 142.24 28.575 0)
       (effects (font (size 1.27 1.27) italic) (justify left) hide)
     )
@@
       (effects (font (size 1.27 1.27)) (justify left))
     )
-    (property "Footprint" "Package_TO_SOT_THT:TO-92_Inline" (id 2) (at 201.93 28.575 0)
+    (property "Footprint" "Package_TO_SOT_THT:TO-92_Inline_Wide" (id 2) (at 201.93 28.575 0)
       (effects (font (size 1.27 1.27) italic) (justify left) hide)
     )
@@
       (effects (font (size 1.27 1.27)) (justify left))
     )
-    (property "Footprint" "Package_TO_SOT_THT:TO-92_Inline" (id 2) (at 262.89 28.575 0)
+    (property "Footprint" "Package_TO_SOT_THT:TO-92_Inline_Wide" (id 2) (at 262.89 28.575 0)
       (effects (font (size 1.27 1.27) italic) (justify left) hide)
     )
@@
       (effects (font (size 1.27 1.27)) (justify left))
     )
-    (property "Footprint" "Package_TO_SOT_THT:TO-92_Inline" (id 2) (at 142.24 79.375 0)
+    (property "Footprint" "Package_TO_SOT_THT:TO-92_Inline_Wide" (id 2) (at 142.24 79.375 0)
       (effects (font (size 1.27 1.27) italic) (justify left) hide)
     )
@@
       (effects (font (size 1.27 1.27)) (justify left))
     )
-    (property "Footprint" "Package_TO_SOT_THT:TO-92_Inline" (id 2) (at 201.93 79.375 0)
+    (property "Footprint" "Package_TO_SOT_THT:TO-92_Inline_Wide" (id 2) (at 201.93 79.375 0)
       (effects (font (size 1.27 1.27) italic) (justify left) hide)
     )
@@
       (effects (font (size 1.27 1.27)) (justify left))
     )
-    (property "Footprint" "Package_TO_SOT_THT:TO-92_Inline" (id 2) (at 262.89 79.375 0)
-      (effects (font (size 1.27 1.27) italic) (justify left) hide)
-    )
+    (property "Footprint" "Package_TO_SOT_THT:TO-92_Inline_Wide" (id 2) (at 262.89 79.375 0)
+      (effects (font (size 1.27 1.27) italic) (justify left) hide)
+    )

Commit message: WIP
Parts:
- removed C5, C7: 10n, Capacitor_THT:C_Rect_L7.0mm_W2.5mm_P5.00mm, symbol Device:C
- removed Q18, Q22, Q6: MPSA42, Package_TO_SOT_THT:TO-92_Inline_Wide, symbol Transistor_BJT:MPSA42
- removed Q20, Q24: KSP92BU, Package_TO_SOT_THT:TO-92_Inline_Wide, symbol Transistor_BJT:MPSA92
- removed R12: 11k 1%, Resistor_THT:R_Axial_DIN0207_L6.3mm_D2.5mm_P10.16mm_Horizontal, symbol Device:R
- removed R34, R43: 11k, Resistor_THT:R_Axial_DIN0207_L6.3mm_D2.5mm_P10.16mm_Horizontal, symbol Device:R
- removed R37, R46: 4k42, Resistor_THT:R_Axial_DIN0207_L6.3mm_D2.5mm_P10.16mm_Horizontal, symbol Device:R
- removed R38, R41, R47, R49: 220k, Resistor_THT:R_Axial_DIN0207_L6.3mm_D2.5mm_P10.16mm_Horizontal, symbol Device:R
- C1: footprint Capacitor_THT:CP_Radial_D8.0mm_P3.80mm -> Capacitor_SMD:C_1812_4532Metric
- C2, C3, C4, C6: footprint Capacitor_THT:C_Rect_L7.0mm_W2.5mm_P5.00mm -> Capacitor_SMD:C_0805_2012Metric
- Q1, Q10, Q11, Q12, Q15, Q16, Q17, Q2, Q21, Q3, Q4, Q5, Q7, Q8, Q9: footprint Package_TO_SOT_THT:TO-92_Inline_Wide -> Package_TO_SOT_SMD:SOT-23; symbol Transistor_BJT:MPSA42 -> Device:Q_NPN_BEC
- Q13, Q14, Q19, Q23: footprint Package_TO_SOT_THT:TO-92_Inline_Wide -> Package_TO_SOT_SMD:SOT-23; symbol Transistor_BJT:MPSA92 -> Device:Q_PNP_BEC
- R1, R10, R11, R13, R14, R15, R16, R17, R18, R19, R2, R20, R21, R22, R23, R24, R25, R26, R27, R28, R29, R3, R30, R31, R32, R33, R35, R36, R39, R4, R40, R42, R44, R45, R48, R5, R6, R7, R8, R9: footprint Resistor_THT:R_Axial_DIN0207_L6.3mm_D2.5mm_P10.16mm_Horizontal -> Resistor_SMD:R_0805_2012Metric
Connections:
- net CA0: now also Q1.1 (B); no longer Q1.2 (B)
- net CA1: now also Q4.1 (B); no longer Q4.2 (B)
- net CA2: now also Q7.1 (B); no longer Q7.2 (B)
- net CA3: now also Q11.1 (B); no longer Q11.2 (B)
- net CA4: now also Q15.1 (B); no longer Q15.2 (B)
- net CA5: now also Q2.1 (B); no longer Q2.2 (B)
- net CA6: now also Q5.1 (B); no longer Q5.2 (B)
- net CA7: now also Q8.1 (B); no longer Q8.2 (B)
- net CA8: now also Q12.1 (B); no longer Q12.2 (B)
- net CA9: now also Q16.1 (B); no longer Q16.2 (B)
- net GND: now also Q10.2 (E), Q17.2 (E), Q21.2 (E), Q9.2 (E); no longer Q10.1 (E), Q17.1 (E), Q21.1 (E), Q9.1 (E)
- net HT: now also Q13.2 (E), Q14.2 (E), Q19.2 (E), Q23.2 (E); no longer Q13.1 (E), Q14.1 (E), Q19.1 (E), Q23.1 (E)
- net S_UN_A: now also Q3.1 (B); no longer Q3.2 (B)
- net at R3.1: now also Q1.2 (E); no longer Q1.1 (E)
- net at R7.1: now also Q3.2 (E); no longer Q3.1 (E)
- net at R17.2: now also Q9.1 (B); no longer Q9.2 (B)
- net at C2.2, R21.2, R22.1: now also Q13.1 (B); no longer Q13.2 (B)
- net at R33.2: now also Q17.1 (B); no longer Q17.2 (B)
- net at C4.2, R35.2, R36.1: now also Q19.1 (B); no longer Q19.2 (B)
- net at R42.2: now also Q21.1 (B); no longer Q21.2 (B)
- net at C6.2, R44.2, R45.1: now also Q23.1 (B); no longer Q23.2 (B)
- net at R18.2: now also Q10.1 (B); no longer Q10.2 (B)
- net at C3.2, R23.2, R24.1: now also Q14.1 (B); no longer Q14.2 (B)
- net at R10.1: now also Q4.2 (E); no longer Q4.1 (E)
- net at R15.1: now also Q7.2 (E); no longer Q7.1 (E)
- net at R25.1: now also Q11.2 (E); no longer Q11.1 (E)
- net at R31.1: now also Q15.2 (E); no longer Q15.1 (E)
- net at R32.1: now also Q16.2 (E); no longer Q16.1 (E)
- net at R26.1: now also Q12.2 (E); no longer Q12.1 (E)
- net at R16.1: now also Q8.2 (E); no longer Q8.1 (E)
- net at R11.1: now also Q5.2 (E); no longer Q5.1 (E)
- net at R4.1: now also Q2.2 (E); no longer Q2.1 (E)
Other:
- moved on the sheet: C6, R42, R44, R45, R48
