File: Oscillator_and_Multiplexing.kicad_sch (KiCad schematic)
At the start: 18 parts, among them U15 74HC4060, U16 4028, U17 74LS151, U18 74LS151, U19 74LS151, U20 4028, U21 74LS151, U3 74LS14, U4 74LS109, U6 74LS08, U7 74LS393, Y1 32.768 kHz - 12.5pF

Commit message: WIP
Parts:
- C34, C35: footprint Capacitor_THT:C_Disc_D5.1mm_W3.2mm_P5.00mm -> Capacitor_SMD:C_0805_2012Metric
- R59, R60, R61: footprint Resistor_THT:R_Axial_DIN0207_L6.3mm_D2.5mm_P10.16mm_Horizontal -> Resistor_SMD:R_0805_2012Metric
Connections:
- net AN5: no longer names the net of U16.1 (S4)
- net AN6: no longer names the net of U16.6 (S5)
- no-connect marks 20 -> 22
Changed lines of the file:
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@@
   (no_connect (at 67.31 44.45))
   (no_connect (at 67.31 34.29))
+  (no_connect (at 148.59 63.5))
+  (no_connect (at 148.59 60.96))
   (no_connect (at 113.03 31.75))
   (no_connect (at 152.4 104.14))
@@
     (stroke (width 0) (type default) (color 0 0 0 0))
   )
+  (wire (pts (xy 148.844 55.88) (xy 148.59 55.88))
+    (stroke (width 0) (type default) (color 0 0 0 0))
+  )
   (wire (pts (xy 100.33 147.32) (xy 107.95 147.32))
     (stroke (width 0) (type default) (color 0 0 0 0))
@@
     (stroke (width 0) (type default) (color 0 0 0 0))
   )
+  (wire (pts (xy 148.844 50.8) (xy 148.59 50.8))
+    (stroke (width 0) (type default) (color 0 0 0 0))
+  )
   (wire (pts (xy 113.03 24.13) (xy 116.84 24.13))
     (stroke (width 0) (type default) (color 0 0 0 0))
@@
     (stroke (width 0) (type default) (color 0 0 0 0))
   )
+  (wire (pts (xy 148.844 58.42) (xy 148.59 58.42))
+    (stroke (width 0) (type default) (color 0 0 0 0))
+  )
   (wire (pts (xy 77.47 24.13) (xy 77.47 31.75))
     (stroke (width 0) (type default) (color 0 0 0 0))
@@
   )
   (wire (pts (xy 163.83 134.62) (xy 163.83 119.38))
+    (stroke (width 0) (type default) (color 0 0 0 0))
+  )
+  (wire (pts (xy 148.844 53.34) (xy 148.59 53.34))
     (stroke (width 0) (type default) (color 0 0 0 0))
   )
@@
     )
   )
-  (global_label "AN5" (shape input) (at 148.59 60.96 0) (fields_autoplaced)
-    (effects (font (size 1.27 1.27)) (justify left))
-    (property "Intersheet References" "${INTERSHEET_REFS}" (id 0) (at 0 0 0)
-      (effects (font (size 1.27 1.27)) hide)
-    )
-  )
   (global_label "CA5" (shape input) (at 266.7 58.42 0) (fields_autoplaced)
     (effects (font (size 1.27 1.27)) (justify left))
@@
     )
   )
-  (global_label "AN3" (shape input) (at 148.59 55.88 0) (fields_autoplaced)
-    (effects (font (size 1.27 1.27)) (justify left))
-    (property "Intersheet References" "${INTERSHEET_REFS}" (id 0) (at 0 0 0)
+  (global_label "AN3" (shape input) (at 148.844 55.88 0) (fields_autoplaced)
+    (effects (font (size 1.27 1.27)) (justify left))
+    (property "Intersheet References" "${INTERSHEET_REFS}" (id 0) (at 0.254 0 0)
       (effects (font (size 1.27 1.27)) hide)
     )
@@
     )
   )
-  (global_label "AN6" (shape input) (at 148.59 63.5 0) (fields_autoplaced)
-    (effects (font (size 1.27 1.27)) (justify left))
-    (property "Intersheet References" "${INTERSHEET_REFS}" (id 0) (at 0 0 0)
-      (effects (font (size 1.27 1.27)) hide)
-    )
-  )
   (global_label "S_DE_A" (shape input) (at 127 111.76 180) (fields_autoplaced)
     (effects (font (size 1.27 1.27)) (justify right))
@@
     )
   )
-  (global_label "AN1" (shape input) (at 148.59 50.8 0) (fields_autoplaced)
-    (effects (font (size 1.27 1.27)) (justify left))
-    (property "Intersheet References" "${INTERSHEET_REFS}" (id 0) (at 0 0 0)
+  (global_label "AN1" (shape input) (at 148.844 50.8 0) (fields_autoplaced)
+    (effects (font (size 1.27 1.27)) (justify left))
+    (property "Intersheet References" "${INTERSHEET_REFS}" (id 0) (at 0.254 0 0)
       (effects (font (size 1.27 1.27)) hide)
     )
@@
     )
   )
-  (global_label "AN2" (shape input) (at 148.59 53.34 0) (fields_autoplaced)
-    (effects (font (size 1.27 1.27)) (justify left))
-    (property "Intersheet References" "${INTERSHEET_REFS}" (id 0) (at 0 0 0)
-      (effects (font (size 1.27 1.27)) hide)
-    )
-  )
-  (global_label "AN4" (shape input) (at 148.59 58.42 0) (fields_autoplaced)
-    (effects (font (size 1.27 1.27)) (justify left))
-    (property "Intersheet References" "${INTERSHEET_REFS}" (id 0) (at 0 0 0)
+  (global_label "AN2" (shape input) (at 148.844 53.34 0) (fields_autoplaced)
+    (effects (font (size 1.27 1.27)) (justify left))
+    (property "Intersheet References" "${INTERSHEET_REFS}" (id 0) (at 0.254 0 0)
+      (effects (font (size 1.27 1.27)) hide)
+    )
+  )
+  (global_label "AN4" (shape input) (at 148.844 58.42 0) (fields_autoplaced)
+    (effects (font (size 1.27 1.27)) (justify left))
+    (property "Intersheet References" "${INTERSHEET_REFS}" (id 0) (at 0.254 0 0)
       (effects (font (size 1.27 1.27)) hide)
     )
@@
       (effects (font (size 1.27 1.27)) (justify left))
     )
-    (property "Footprint" "Resistor_THT:R_Axial_DIN0207_L6.3mm_D2.5mm_P10.16mm_Horizontal" (id 2) (at 38.608 50.8 90)
+    (property "Footprint" "Resistor_SMD:R_0805_2012Metric" (id 2) (at 38.608 50.8 90)
       (effects (font (size 1.27 1.27)) hide)
     )
@@
       (effects (font (size 1.27 1.27)) (justify left))
     )
-    (property "Footprint" "Capacitor_THT:C_Disc_D5.1mm_W3.2mm_P5.00mm" (id 2) (at 35.8648 67.31 0)
+    (property "Footprint" "Capacitor_SMD:C_0805_2012Metric" (id 2) (at 35.8648 67.31 0)
       (effects (font (size 1.27 1.27)) hide)
     )
@@
   (symbol (lib_id "Device:Crystal") (at 30.48 57.15 0) (mirror y) (unit 1)
     (in_bom yes) (on_board yes)
-    (property "Reference" "Y1" (id 0) (at 30.48 50.3428 0))
-    (property "Value" "32.768 kHz - 12.5pF" (id 1) (at 30.48 52.6542 0))
+    (property "Reference" "Y1" (id 0) (at 28.321 52.578 0))
+    (property "Value" "32.768 kHz - 12.5pF" (id 1) (at 30.353 41.402 0))
     (property "Footprint" "Crystal:Crystal_C38-LF_D3.0mm_L8.0mm_Vertical" (id 2) (at 30.48 57.15 0)
       (effects (font (size 1.27 1.27)) hide)
@@
       (effects (font (size 1.27 1.27)) (justify left))
     )
-    (property "Footprint" "Capacitor_THT:C_Disc_D5.1mm_W3.2mm_P5.00mm" (id 2) (at 23.1648 67.31 0)
+    (property "Footprint" "Capacitor_SMD:C_0805_2012Metric" (id 2) (at 23.1648 67.31 0)
       (effects (font (size 1.27 1.27)) hide)
     )
@@
       (effects (font (size 1.27 1.27)) (justify right))
     )
-    (property "Footprint" "Resistor_THT:R_Axial_DIN0207_L6.3mm_D2.5mm_P10.16mm_Horizontal" (id 2) (at 22.352 50.8 90)
+    (property "Footprint" "Resistor_SMD:R_0805_2012Metric" (id 2) (at 22.352 50.8 90)
       (effects (font (size 1.27 1.27)) hide)
     )
@@
       (effects (font (size 1.27 1.27)) (justify right))
     )
-    (property "Footprint" "Resistor_THT:R_Axial_DIN0207_L6.3mm_D2.5mm_P10.16mm_Horizontal" (id 2) (at 71.12 159.512 90)
-      (effects (font (size 1.27 1.27)) hide)
-    )
+    (property "Footprint" "Resistor_SMD:R_0805_2012Metric" (id 2) (at 71.12 159.512 90)
+      (effects (font (size 1.27 1.27)) hide)
+    )
