File: Oscillator_and_Multiplexing.kicad_sch (KiCad schematic)
At the start: 18 parts, among them U15 74HC4060, U16 4028, U17 74LS151, U18 74LS151, U19 74LS151, U20 4028, U21 74LS151, U3 74LS14, U4 74LS109, U6 74LS08, U7 74LS393, Y1 32.768 kHz - 12.5pF

Commit message: layout started
Parts:
- renumbered C33 to C34, C34 to C35, C35 to C36
