File: NixieClock.kicad_pcb (KiCad board)
At the start: 2 copper layers, 170 x 132 mm, 147 parts, among them J1 Barrel_Jack, Q1 MPSA42, Q10 MPSA42, Q11 MPSA42, Q12 MPSA42, Q13 KSP92BU, Q14 KSP92BU, Q15 MPSA42, Q16 MPSA42, Q17 MPSA42, Q19 KSP92BU, Q2 MPSA42, Q21 MPSA42, Q23 KSP92BU, Q25 KSP2907A, Q26 IRF644, Q3 MPSA42, Q4 MPSA42, Q5 MPSA42, Q7 MPSA42, Q8 MPSA42, Q9 MPSA42, SW1 PB400EEQX, SW3 SW_Push, SW4 SW_Push, U1 L7805, U10 74LS160, U11 74LS160, U12 74LS160, U13 74LS160, U14 74LS160, U15 74HC4060, U16 4028, U17 74LS151, U18 74LS151, U19 74LS151, U2 MC34063AP, U20 4028, U21 74LS151, U3 74LS14, U4 74LS109, U5 74LS10, U6 74LS08, U7 74LS393, U8 74LS20, U9 74LS160, Y1 32.768 kHz - 12.5pF

Commit message: DRC 0k
Parts:
- moved R39 13.2 mm to (180.1, 144.8)
Routing:
- net S_UN_A: track 160.5 -> 149.5 mm
- net +5V: track 806.9 -> 803.2 mm
- net AN1: track 108.2 -> 106.4 mm
- net AN2: track 94.4 -> 92.7 mm, vias 2 -> 1
- net CA5: track 74.5 -> 73.2 mm
- net CA4: track 157.1 -> 155.8 mm
- net CA3: track 161.9 -> 160.8 mm
- net Net-(R57-Pad2): track 109.3 -> 108.3 mm
- net AN4: track 57.7 -> 56.7 mm
- net KDP: track 99.8 -> 99.0 mm
- net Net-(C2-Pad2): track 6.37 -> 5.83 mm
